Commit message: initial commit

File: source/instinctlab/instinctlab/tasks/parkour/urdf/g1_29dof_torsoBase_popsicle_with_shoe_copy.urdf (robot description, URDF)
Before this commit: robot g1, 40 links, 39 joints
Links:
- link left_ankle_roll_link: geometry collision mesh filename=../../../assets/resources/unitree_g1/meshes/left_ankle_roll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; visual mesh filename=../../../assets/resources/unitree_g1/meshes/left_ankle_roll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
- link right_ankle_roll_link: geometry collision mesh filename=../../../assets/resources/unitree_g1/meshes/right_ankle_rol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; visual mesh filename=../../../assets/resources/unitree_g1/meshes/right_ankle_rol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
